File: controller/controller.sch (KiCad schematic (older format))
At the start: 23 parts, among them Q1 Q_NJFET_GDS, U1 74HC595

Commit message: Clean up gang controller code
Parts:
- R3: footprint (none) -> Resistors_THT:R_Axial_DIN0204_L3.6mm_D1.6mm_P5.08mm_Horizontal
Changed lines of the file:
@@
 F 0 "R3" H 2668 2146 50  0000 L CNN
 F 1 "1M" H 2668 2055 50  0000 L CNN
-F 2 "" V 2640 2090 50  0001 C CNN
+F 2 "Resistors_THT:R_Axial_DIN0204_L3.6mm_D1.6mm_P5.08mm_Horizontal" V 2640 2090 50  0001 C CNN
 F 3 "~" H 2600 2100 50  0001 C CNN
 	1    2600 2100
